Commit message: Push_preHW03
HW01 man + opt done
HW02 man done
HW03 - extra files not added, notes to hw added

File: robotics_labs-main/src/robotics_toolbox/robots/robot_hw.urdf (robot description, URDF)
Before this commit: robot simple_robot, 2 links, 1 joints
Links:
- removed link base_link
- added link base; visual box size=0.3 0.3 0.3
- added link cylinder_1; visual cylinder length=0.5 radius=0.05
- added link cylinder_2; visual cylinder length=0.25 radius=0.05
- added link cylinder_3; visual cylinder length=0.25 radius=0.05
- added link cylinder_4; visual cylinder length=0.25 radius=0.05
- added link sphere_1; visual sphere radius=0.06
- added link sphere_2; visual sphere radius=0.06
Joints:
- removed joint joint0
- added joint fixed_sphere_1: type fixed, parent cylinder_1, child sphere_1, origin xyz=0 0 0.5 rpy=0 0 0
- added joint fixed_sphere_2: type fixed, parent cylinder_3, child sphere_2, origin xyz=0 0 0.25 rpy=0 0 0
- added joint joint_X: type revolute, parent sphere_1, child cylinder_2, origin xyz=0 0 0 rpy=0 0 0, axis 1 0 0, limit lower=-3.14 upper=3.14 effort=10 velocity=1.0
- added joint joint_X_2: type revolute, parent sphere_2, child cylinder_4, origin xyz=0 0 0 rpy=0 0 0, axis 1 0 0, limit lower=-3.14 upper=3.14 effort=10 velocity=1.0
- added joint joint_Z: type revolute, parent base, child cylinder_1, origin xyz=0 0 0.15 rpy=0 0 0, axis 0 0 1, limit lower=-3.14 upper=3.14 effort=10 velocity=1.0
- added joint joint_Z_2: type revolute, parent cylinder_2, child cylinder_3, origin xyz=0 0 0.25 rpy=0 0 0, axis 0 0 1, limit lower=-3.14 upper=3.14 effort=10 velocity=1.0
- added joint joint_fixed_effector: type fixed, parent cylinder_4, child end_effector, origin xyz=0 0 0.25 rpy=0 0 0
